File: hardware/mx_thru_hole_reversible/kbd.kicad_pcb (KiCad board)
At the start: 2 copper layers, 135.7 x 107.4 mm, 76 parts, among them J1 Conn_01x12_MountingPin, J2 Conn_01x12_MountingPin, SW00 SW_Push, SW01 SW_Push, SW02 SW_Push, SW03 SW_Push, SW04 SW_Push, SW05 SW_Push, SW10 SW_Push, SW11 SW_Push, SW12 SW_Push, SW13 SW_Push, SW14 SW_Push, SW15 SW_Push, SW20 SW_Push, SW21 SW_Push, SW22 SW_Push, SW23 SW_Push, SW24 SW_Push, SW25 SW_Push, SW30 SW_Push, SW31 SW_Push, SW32 SW_Push, SW33 SW_Push, SW34 SW_Push, SW35 SW_Push, SW36 SW_Push, SW37 SW_Push, U1 CH582, U2 74HC165, U4 74HC165

Commit message: Clean up
Parts:
- moved RN2 47.9 mm to (185.1, 114.5), turned to 0 degrees
- moved RN1 47.0 mm to (183.3, 114.5), turned to 180 degrees
- moved U2 37.3 mm to (177.2, 115.1), turned to 0 degrees
- moved U4 33.8 mm to (172.2, 115.1), turned to 180 degrees
- moved JP2 8.11 mm to (185.6, 124.3)
- moved R1 1.33 mm to (174.7, 45.5)
Routing:
- net DS: track 65.0 -> 18.4 mm
- net COL1: track 167.3 -> 208.7 mm
- net MISO: track 95.4 -> 55.6 mm
- net COL3: track 144.1 -> 182.6 mm, vias 2 -> 3
- net COL0: track 194.7 -> 232.9 mm
- net COL2: track 161.5 -> 198.3 mm
- net COL4: track 131.3 -> 163.5 mm, vias 2 -> 3
- net +3V3: track 132.0 -> 102.8 mm
- net SCK0: track 99.3 -> 71.8 mm
- net COL5: track 128.1 -> 152.8 mm
- net SCS: track 99.3 -> 75.5 mm
- net COL7: track 58.1 -> 37.5 mm
- net COL6: track 34.8 -> 45.7 mm, vias 2 -> 3
- net ROW3: track 211.7 -> 207.3 mm, vias 3 -> 2
- net GND: track 125.0 -> 129.1 mm, vias 29 -> 27
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Other:
- board size 135.7 x 107.4 mm -> 146.1 x 106.6 mm
