File: hardware/mx_thru_hole_reversible/kbd.kicad_sch (KiCad schematic)
At the start: 76 parts, among them J1 Conn_01x12_MountingPin, J2 Conn_01x12_MountingPin, SW00 SW_Push, SW01 SW_Push, SW02 SW_Push, SW03 SW_Push, SW04 SW_Push, SW05 SW_Push, SW10 SW_Push, SW11 SW_Push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

Commit message: Clean up
Other:
- moved on the sheet: RN2, U2

Commit message: Cleaned up footprint library, added new design, updated python script
Other:
- moved on the sheet: RN1, RN2
