File: hardware/choc_v1_socket_reversible_165_595/choc_v1_socket_reversible_165_595.kicad_pcb (KiCad board)
At the start: 2 copper layers, 3.4 x 3 mm, 70 parts, among them SW00 SW_Push, SW01 SW_Push, SW02 SW_Push, SW03 SW_Push, SW04 SW_Push, SW05 SW_Push, SW10 SW_Push, SW11 SW_Push, SW12 SW_Push, SW13 SW_Push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

Commit message: Finished layout
Parts:
- D0, D1, D2, D3, D4, D5, D6, JP1, J_LEFT1, R1, R2, RN_LEFT1, SR_LEFT1: moved to B.Cu
- moved SW05 293.2 mm to (155.0, 53.5)
- moved SW04 272.6 mm to (136.0, 51.0)
- moved SW15 270.2 mm to (155.0, 70.5)
- moved SW36 259.1 mm to (178.8, 130.8), turned to -30 degrees
- moved SW26 257.4 mm to (157.9, 125.8), turned to -23 degrees
- moved SW03 252.6 mm to (117.0, 48.5)
- moved SW25 251.4 mm to (155.0, 87.5)
- moved SW14 251.2 mm to (136.0, 68.0)
- moved RN_LEFT1 250.5 mm to (187.8, 112.0)
- moved RN_RIGHT1 244.5 mm to (186.0, 112.0), turned to 180 degrees
- moved JP1 244.2 mm to (175.6, 54.0)
- moved JP2 241.9 mm to (186.3, 125.5)
- moved LED36 234.7 mm to (181.2, 126.7), turned to -30 degrees
- moved SW24 234.5 mm to (136.0, 85.0)
- moved SW35 233.9 mm to (155.0, 104.5)
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Connections:
- LED01 pad 3: Net-(LED00-DOUT) -> Net-(LED01-DIN)
- LED02 pad 1: Net-(LED02-DOUT) -> Net-(LED01-DIN)
- LED03 pad 1: Net-(LED02-DIN) -> Net-(LED03-DOUT)
- LED04 pad 1: Net-(LED04-DOUT) -> Net-(LED03-DIN)
- LED05 pad 1: Net-(LED04-DIN) -> Net-(LED05-DOUT)
- LED12 pad 1: Net-(LED12-DOUT) -> Net-(LED02-DIN)
- LED12 pad 3: Net-(LED02-DOUT) -> Net-(LED12-DIN)
- LED13 pad 1: Net-(LED03-DIN) -> Net-(LED13-DOUT)
- LED13 pad 3: Net-(LED13-DIN) -> Net-(LED03-DOUT)
- LED14 pad 1: Net-(LED14-DOUT) -> Net-(LED04-DIN)
- LED14 pad 3: Net-(LED04-DOUT) -> Net-(LED14-DIN)
- LED15 pad 1: Net-(LED05-DIN) -> Net-(LED15-DOUT)
- LED15 pad 3: Net-(LED15-DIN) -> Net-(LED05-DOUT)
- LED22 pad 1: Net-(LED22-DOUT) -> Net-(LED12-DIN)
- LED22 pad 3: Net-(LED12-DOUT) -> Net-(LED22-DIN)
- LED23 pad 1: Net-(LED13-DIN) -> Net-(LED23-DOUT)
- LED23 pad 3: Net-(LED23-DIN) -> Net-(LED13-DOUT)
- LED24 pad 1: Net-(LED24-DOUT) -> Net-(LED14-DIN)
- LED24 pad 3: Net-(LED14-DOUT) -> Net-(LED24-DIN)
- LED25 pad 1: Net-(LED15-DIN) -> Net-(LED25-DOUT)
- LED25 pad 3: Net-(LED25-DIN) -> Net-(LED15-DOUT)
- LED26 pad 3: Net-(LED26-DIN) -> Net-(LED00-DOUT)
- LED30 pad 3: Net-(LED26-DIN) -> Net-(LED30-DIN)
- LED31 pad 1: Net-(LED31-DOUT) -> Net-(LED30-DIN)
- LED32 pad 1: Net-(LED31-DOUT) -> Net-(LED22-DIN)
- LED32 pad 3: Net-(LED22-DOUT) -> Net-(LED32-DIN)
- LED33 pad 1: Net-(LED23-DIN) -> Net-(LED32-DIN)
- LED33 pad 3: Net-(LED33-DIN) -> Net-(LED23-DOUT)
- LED34 pad 1: Net-(LED33-DIN) -> Net-(LED24-DIN)
- LED34 pad 3: Net-(LED24-DOUT) -> Net-(LED34-DIN)
- LED35 pad 1: Net-(LED25-DIN) -> Net-(LED34-DIN)
- LED35 pad 3: Net-(LED35-DIN) -> Net-(LED25-DOUT)
- R2 pad 1: Net-(LED35-DIN) -> Net-(LED05-DIN)
- RN_LEFT1 pad 1: COL4 -> COL7
- RN_LEFT1 pad 2: COL3 -> COL6
- RN_LEFT1 pad 3: COL5 -> COL0
- RN_LEFT1 pad 4: COL2 -> COL1
- RN_LEFT1 pad 5: COL6 -> COL2
- RN_LEFT1 pad 6: COL1 -> COL3
- RN_LEFT1 pad 7: COL7 -> COL4
- RN_LEFT1 pad 8: COL0 -> COL5
- RN_RIGHT1 pad 1: COL4 -> COL7
- RN_RIGHT1 pad 2: COL3 -> COL6
- RN_RIGHT1 pad 3: COL5 -> COL0
- RN_RIGHT1 pad 4: COL2 -> COL1
- RN_RIGHT1 pad 5: COL6 -> COL2
- RN_RIGHT1 pad 6: COL1 -> COL3
- RN_RIGHT1 pad 7: COL7 -> COL4
- RN_RIGHT1 pad 8: COL0 -> COL5
- SR_LEFT1 pad 11: COL0 -> COL5
- SR_LEFT1 pad 12: COL1 -> COL3
- SR_LEFT1 pad 13: COL2 -> COL1
- SR_LEFT1 pad 14: COL3 -> COL6
- SR_LEFT1 pad 3: COL4 -> COL7
- SR_LEFT1 pad 4: COL5 -> COL0
- SR_LEFT1 pad 5: COL6 -> COL2
- SR_LEFT1 pad 6: COL7 -> COL4
- SR_RIGHT1 pad 11: COL0 -> COL5
- SR_RIGHT1 pad 12: COL1 -> COL3
- SR_RIGHT1 pad 13: COL2 -> COL1
- SR_RIGHT1 pad 14: COL3 -> COL6
- SR_RIGHT1 pad 3: COL4 -> COL7
- SR_RIGHT1 pad 4: COL5 -> COL0
- SR_RIGHT1 pad 5: COL6 -> COL2
- SR_RIGHT1 pad 6: COL7 -> COL4
- SW20 pad 1: Net-(D0C-K) -> Net-(D0D-K)
- SW21 pad 1: Net-(D1C-K) -> Net-(D1D-K)
- SW22 pad 1: Net-(D2C-K) -> Net-(D2D-K)
- SW23 pad 1: Net-(D3C-K) -> Net-(D3D-K)
- SW24 pad 1: Net-(D4C-K) -> Net-(D4D-K)
- SW25 pad 1: Net-(D5C-K) -> Net-(D5D-K)
- SW26 pad 1: Net-(D6C-K) -> Net-(D6D-K)
- SW30 pad 1: Net-(D0D-K) -> Net-(D0C-K)
- SW31 pad 1: Net-(D1D-K) -> Net-(D1C-K)
- SW32 pad 1: Net-(D2D-K) -> Net-(D2C-K)
- SW33 pad 1: Net-(D3D-K) -> Net-(D3C-K)
- SW34 pad 1: Net-(D4D-K) -> Net-(D4C-K)
- SW35 pad 1: Net-(D5D-K) -> Net-(D5C-K)
- SW36 pad 1: Net-(D6D-K) -> Net-(D6C-K)
Routing:
- net +5V: track 0.00 -> 629.9 mm, vias 0 -> 27
- net ROW2: track 0.00 -> 267.0 mm, vias 0 -> 8
- net ROW3: track 0.00 -> 263.7 mm, vias 0 -> 9
- net ROW1: track 0.00 -> 209.6 mm, vias 0 -> 7
- net ROW0: track 0.00 -> 203.7 mm, vias 0 -> 7
- net Net-(LED00-DOUT): track 0.00 -> 164.6 mm, vias 0 -> 3
- net COL0: track 0.00 -> 145.3 mm, vias 0 -> 3
- net COL1: track 0.00 -> 125.4 mm, vias 0 -> 3
- net COL2: track 0.00 -> 106.7 mm, vias 0 -> 3
- net +3V3: track 0.00 -> 91.3 mm, vias 0 -> 3
- net LED_R: track 0.00 -> 90.4 mm, vias 0 -> 2
- net COL3: track 0.00 -> 87.8 mm, vias 0 -> 3
- net SCS: track 0.00 -> 69.7 mm, vias 0 -> 2
- net COL4: track 0.00 -> 68.7 mm, vias 0 -> 3
- net Net-(D1A-K): track 0.00 -> 64.3 mm, vias 0 -> 2
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- added copper zone on B.Cu, net GND
- added copper zone on F.Cu, net GND
Other:
- board size 3.4 x 3 mm -> 143.8 x 106.1 mm

Commit message: Updated schematic to use 0805 ressitor and 1x12 FFC socket
Parts:
- removed RN_LEFT1, RN_RIGHT1: R_Pack08, Resistor_SMD:R_Array_Convex_8x0602
- added R_L0: R_US, Resistor_SMD:R_0805_2012Metric_Pad1.20x1.40mm_HandSolder, F.Cu at (-23.1, 54.0)
- added R_L1: R_US, Resistor_SMD:R_0805_2012Metric_Pad1.20x1.40mm_HandSolder, F.Cu at (-23.1, 57.0)
- added R_L2: R_US, Resistor_SMD:R_0805_2012Metric_Pad1.20x1.40mm_HandSolder, F.Cu at (-23.1, 60.0)
- added R_L3: R_US, Resistor_SMD:R_0805_2012Metric_Pad1.20x1.40mm_HandSolder, F.Cu at (-23.1, 62.9)
- added R_L4: R_US, Resistor_SMD:R_0805_2012Metric_Pad1.20x1.40mm_HandSolder, F.Cu at (-23.1, 65.8)
- added R_L5: R_US, Resistor_SMD:R_0805_2012Metric_Pad1.20x1.40mm_HandSolder, F.Cu at (-23.1, 68.8)
- added R_L6: R_US, Resistor_SMD:R_0805_2012Metric_Pad1.20x1.40mm_HandSolder, F.Cu at (-18.4, 54.0)
- added R_L7: R_US, Resistor_SMD:R_0805_2012Metric_Pad1.20x1.40mm_HandSolder, F.Cu at (-18.4, 57.0)
- added R_R0: R_US, Resistor_SMD:R_0805_2012Metric_Pad1.20x1.40mm_HandSolder, F.Cu at (-18.4, 60.0)
- added R_R1: R_US, Resistor_SMD:R_0805_2012Metric_Pad1.20x1.40mm_HandSolder, F.Cu at (-18.4, 62.9)
- added R_R2: R_US, Resistor_SMD:R_0805_2012Metric_Pad1.20x1.40mm_HandSolder, F.Cu at (-18.4, 65.8)
- added R_R3: R_US, Resistor_SMD:R_0805_2012Metric_Pad1.20x1.40mm_HandSolder, F.Cu at (-18.4, 68.8)
- added R_R4: R_US, Resistor_SMD:R_0805_2012Metric_Pad1.20x1.40mm_HandSolder, F.Cu at (-13.6, 54.0)
- added R_R5: R_US, Resistor_SMD:R_0805_2012Metric_Pad1.20x1.40mm_HandSolder, F.Cu at (-13.6, 57.0)
- added R_R6: R_US, Resistor_SMD:R_0805_2012Metric_Pad1.20x1.40mm_HandSolder, F.Cu at (-13.6, 60.0)
- added R_R7: R_US, Resistor_SMD:R_0805_2012Metric_Pad1.20x1.40mm_HandSolder, F.Cu at (-13.6, 62.9)
- D0, D1, D2, D3, D4, D5, D6, JP1, R1, R2, SR_LEFT1: moved to F.Cu
- J_LEFT1: value Conn_02x12_Odd_Even_MountingPin -> Conn_01x12_MountingPin; footprint Connector_FFC-FPC:Jushuo_AFC07-S24FCA-00_1x24-1MP_P0.50_Horizontal -> Connector_FFC-FPC:JUSHUO_AFA07-S12FCA-00_1x12-1MP_P1.0mm_Horizontal; moved to F.Cu
- J_RIGHT1: value Conn_02x12_Odd_Even_MountingPin -> Conn_01x12_MountingPin; footprint Connector_FFC-FPC:Jushuo_AFC07-S24FCA-00_1x24-1MP_P0.50_Horizontal -> Connector_FFC-FPC:JUSHUO_AFA07-S12FCA-00_1x12-1MP_P1.0mm_Horizontal
- moved SW05 276.0 mm to (-117.0, 100.4)
- moved SW04 255.1 mm to (-117.0, 83.5)
- moved SW15 252.2 mm to (-96.8, 83.5)
- moved SW36 240.0 mm to (-56.5, 83.5), turned to 0 degrees
- moved SW26 238.4 mm to (-76.7, 83.5), turned to 0 degrees
- moved SW03 234.7 mm to (-117.0, 66.7)
- moved SW14 232.9 mm to (-96.8, 66.7)
- moved SW25 232.6 mm to (-76.7, 66.7)
- moved JP2 230.6 mm to (-44.3, 122.9)
- moved R1 229.8 mm to (-44.3, 116.7), turned to 0 degrees
- moved R2 228.4 mm to (-44.3, 119.7)
- moved JP1 226.5 mm to (-43.0, 113.5)
- moved LED36 215.8 mm to (-13.6, 33.7), turned to 0 degrees
- moved SW24 215.6 mm to (-76.7, 49.8)
- moved SW02 215.0 mm to (-117.0, 49.8)
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Connections:
- J_LEFT1 pad 10: DS -> +5V
- J_LEFT1 pad 11: ROW1 -> unconnected-(J_LEFT1-Pin_11-Pad11)
- J_LEFT1 pad 12: ROW1 -> GND
- J_LEFT1 pad 2: ROW3 -> ROW2
- J_LEFT1 pad 3: ROW2 -> SCK0
- J_LEFT1 pad 4: ROW2 -> SCS
- J_LEFT1 pad 5: SCK0 -> DS
- J_LEFT1 pad 6: SCK0 -> ROW1
- J_LEFT1 pad 7: SCS -> ROW0
- J_LEFT1 pad 8: SCS -> +3V3
- J_LEFT1 pad 9: DS -> LED_R
- J_RIGHT1 pad 10: +3V3 -> SCK0
- J_RIGHT1 pad 11: ROW0 -> ROW2
- J_RIGHT1 pad 12: ROW0 -> ROW3
- J_RIGHT1 pad 2: GND -> unconnected-(J_RIGHT1-Pin_2-Pad2)
- J_RIGHT1 pad 3: unconnected-(J_RIGHT1-Pin_3-Pad3) -> +5V
- J_RIGHT1 pad 4: unconnected-(J_RIGHT1-Pin_4-Pad4) -> LED_R
- J_RIGHT1 pad 5: +5V -> +3V3
- J_RIGHT1 pad 6: +5V -> ROW0
- J_RIGHT1 pad 7: LED_R -> ROW1
- J_RIGHT1 pad 8: LED_R -> DS
- J_RIGHT1 pad 9: +3V3 -> SCS
Routing:
- net +5V: track 629.9 -> 0.00 mm, vias 27 -> 0
- net ROW2: track 267.0 -> 0.00 mm, vias 8 -> 0
- net ROW3: track 263.7 -> 0.00 mm, vias 9 -> 0
- net ROW1: track 209.6 -> 0.00 mm, vias 7 -> 0
- net ROW0: track 203.7 -> 0.00 mm, vias 7 -> 0
- net Net-(LED00-DOUT): track 164.6 -> 0.00 mm, vias 3 -> 0
- net COL0: track 145.3 -> 0.00 mm, vias 3 -> 0
- net COL1: track 125.4 -> 0.00 mm, vias 3 -> 0
- net COL2: track 106.7 -> 0.00 mm, vias 3 -> 0
- net +3V3: track 91.3 -> 0.00 mm, vias 3 -> 0
- net LED_R: track 90.4 -> 0.00 mm, vias 2 -> 0
- net COL3: track 87.8 -> 0.00 mm, vias 3 -> 0
- net SCS: track 69.7 -> 0.00 mm, vias 2 -> 0
- net COL4: track 68.7 -> 0.00 mm, vias 3 -> 0
- net Net-(D1A-K): track 64.3 -> 0.00 mm, vias 2 -> 0
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- removed copper zone on B.Cu, net GND
- removed copper zone on F.Cu, net GND
Other:
- board size 143.8 x 106.1 mm -> 3.4 x 3 mm

Commit message: Updated connector and resistor for easier SMD soldering
Parts:
- J_LEFT1, J_RIGHT1: value Conn_01x12_MountingPin -> FPC11-X1.0-12AH2.5; footprint Connector_FFC-FPC:JUSHUO_AFA07-S12FCA-00_1x12-1MP_P1.0mm_Horizontal -> easyeda2kicad:FPC-SMD_12P-P1.00_XYECONN_FPC10-S1.0-12AH2.5
- moved R_L0 48.1 mm to (-45.2, 96.8)
- moved R_L1 48.1 mm to (-45.2, 99.8)
- moved R_L4 48.1 mm to (-45.2, 108.6)
- moved R_L5 48.1 mm to (-45.2, 111.6)
- moved R_L6 48.1 mm to (-40.4, 96.8)
- moved R_L7 48.1 mm to (-40.4, 99.8)
- moved R_R2 48.1 mm to (-40.4, 108.6)
- moved R_R3 48.1 mm to (-40.4, 111.6)
- moved R_R4 48.1 mm to (-35.7, 96.8)
- moved R_R5 48.1 mm to (-35.7, 99.8)
- moved R_L3 48.1 mm to (-45.2, 105.7)
- moved R_R1 48.1 mm to (-40.4, 105.7)
- moved R_R7 48.1 mm to (-35.7, 105.7)
- moved R_L2 48.1 mm to (-45.2, 102.7)
- moved R_R0 48.1 mm to (-40.4, 102.7)
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Connections:
- J_LEFT1 pad 1: ROW3 -> GND
- J_LEFT1 pad 10: +5V -> SCK0
- J_LEFT1 pad 11: unconnected-(J_LEFT1-Pin_11-Pad11) -> ROW2
- J_LEFT1 pad 12: GND -> ROW3
- J_LEFT1 pad 2: ROW2 -> unconnected-(J_LEFT1-Pad2)
- J_LEFT1 pad 3: SCK0 -> +5V
- J_LEFT1 pad 4: SCS -> LED_R
- J_LEFT1 pad 5: DS -> +3V3
- J_LEFT1 pad 6: ROW1 -> ROW0
- J_LEFT1 pad 7: ROW0 -> ROW1
- J_LEFT1 pad 8: +3V3 -> DS
- J_LEFT1 pad 9: LED_R -> SCS
- J_RIGHT1 pad 1: GND -> ROW3
- J_RIGHT1 pad 10: SCK0 -> +5V
- J_RIGHT1 pad 11: ROW2 -> unconnected-(J_RIGHT1-Pad11)
- J_RIGHT1 pad 12: ROW3 -> GND
- J_RIGHT1 pad 2: unconnected-(J_RIGHT1-Pin_2-Pad2) -> ROW2
- J_RIGHT1 pad 3: +5V -> SCK0
- J_RIGHT1 pad 4: LED_R -> SCS
- J_RIGHT1 pad 5: +3V3 -> DS
- J_RIGHT1 pad 6: ROW0 -> ROW1
- J_RIGHT1 pad 7: ROW1 -> ROW0
- J_RIGHT1 pad 8: DS -> +3V3
- J_RIGHT1 pad 9: SCS -> LED_R
- R_L0 pad 2: COL7 -> COL0
- R_L1 pad 2: COL6 -> COL1
- R_L2 pad 2: COL0 -> COL2
- R_L3 pad 2: COL1 -> COL3
- R_L4 pad 2: COL2 -> COL4
- R_L5 pad 2: COL3 -> COL5
- R_L6 pad 2: COL4 -> COL6
- R_L7 pad 2: COL5 -> COL7
- R_R0 pad 2: COL7 -> COL0
- R_R1 pad 2: COL6 -> COL1
- R_R2 pad 2: COL0 -> COL2
- R_R3 pad 2: COL1 -> COL3
- R_R4 pad 2: COL2 -> COL4
- R_R5 pad 2: COL3 -> COL5
- R_R6 pad 2: COL4 -> COL6
- R_R7 pad 2: COL5 -> COL7

Commit message: Fixed SER-QH connection
Connections:
- J_LEFT1 pad 10: SCK0 -> DS
- J_LEFT1 pad 8: DS -> SCS
- J_LEFT1 pad 9: SCS -> SCK0
- J_RIGHT1 pad 3: SCK0 -> DS
- J_RIGHT1 pad 4: SCS -> SCK0
- J_RIGHT1 pad 5: DS -> SCS
- SR_LEFT1 pad 7: MISO -> unconnected-(SR_LEFT1-~{Q7}-Pad7)
- SR_LEFT1 pad 9: unconnected-(SR_LEFT1-Q7-Pad9) -> MISO
- SR_RIGHT1 pad 7: DS -> unconnected-(SR_RIGHT1-~{Q7}-Pad7)
- SR_RIGHT1 pad 9: unconnected-(SR_RIGHT1-Q7-Pad9) -> DS
Changed lines of the file:
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@@
 	(net 75 "Net-(LED34-DIN)")
 	(net 76 "COL7")
-	(net 77 "unconnected-(SR_LEFT1-Q7-Pad9)")
+	(net 77 "unconnected-(SR_LEFT1-~{Q7}-Pad7)")
 	(net 78 "MISO")
-	(net 79 "unconnected-(SR_RIGHT1-Q7-Pad9)")
+	(net 79 "unconnected-(SR_RIGHT1-~{Q7}-Pad7)")
 	(net 80 "unconnected-(SR_RIGHT1-DS-Pad10)")
 	(net 81 "unconnected-(U1-B10-Pad8)")
@@
 			(size 0.6 2.5)
 			(layers "F.Cu" "F.Paste" "F.Mask")
-			(net 44 "SCK0")
+			(net 42 "DS")
 			(pinfunction "3")
 			(pintype "unspecified")
@@
 			(size 0.6 2.5)
 			(layers "F.Cu" "F.Paste" "F.Mask")
-			(net 41 "SCS")
+			(net 44 "SCK0")
 			(pinfunction "4")
 			(pintype "unspecified")
@@
 			(size 0.6 2.5)
 			(layers "F.Cu" "F.Paste" "F.Mask")
-			(net 42 "DS")
+			(net 41 "SCS")
 			(pinfunction "5")
 			(pintype "unspecified")
@@
 			(layers "F.Cu" "F.Paste" "F.Mask")
 			(roundrect_rratio 0.25)
-			(net 42 "DS")
+			(net 79 "unconnected-(SR_RIGHT1-~{Q7}-Pad7)")
 			(pinfunction "~{Q7}")
-			(pintype "output")
+			(pintype "output+no_connect")
 		)
 		(pad "8" smd roundrect
@@
 			(layers "F.Cu" "F.Paste" "F.Mask")
 			(roundrect_rratio 0.25)
-			(net 79 "unconnected-(SR_RIGHT1-Q7-Pad9)")
+			(net 42 "DS")
 			(pinfunction "Q7")
-			(pintype "output+no_connect")
+			(pintype "output")
 		)
 		(pad "10" smd roundrect
@@
 			(layers "F.Cu" "F.Paste" "F.Mask")
 			(roundrect_rratio 0.25)
-			(net 78 "MISO")
+			(net 77 "unconnected-(SR_LEFT1-~{Q7}-Pad7)")
 			(pinfunction "~{Q7}")
-			(pintype "output")
+			(pintype "output+no_connect")
 		)
 		(pad "8" smd roundrect
@@
 			(layers "F.Cu" "F.Paste" "F.Mask")
 			(roundrect_rratio 0.25)
-			(net 77 "unconnected-(SR_LEFT1-Q7-Pad9)")
+			(net 78 "MISO")
 			(pinfunction "Q7")
-			(pintype "output+no_connect")
+			(pintype "output")
 		)
 		(pad "10" smd roundrect
@@
 			(size 0.6 2.5)
 			(layers "F.Cu" "F.Paste" "F.Mask")
-			(net 42 "DS")
+			(net 41 "SCS")
 			(pinfunction "8")
 			(pintype "unspecified")
@@
 			(size 0.6 2.5)
 			(layers "F.Cu" "F.Paste" "F.Mask")
-			(net 41 "SCS")
+			(net 44 "SCK0")
 			(pinfunction "9")
 			(pintype "unspecified")
@@
 			(size 0.6 2.5)
 			(layers "F.Cu" "F.Paste" "F.Mask")
-			(net 44 "SCK0")
+			(net 42 "DS")
 			(pinfunction "10")
 			(pintype "unspecified")

Commit message: Fixed Q7-SER connection
Connections:
- SR_RIGHT1 pad 10: unconnected-(SR_RIGHT1-DS-Pad10) -> +3V3
Changed lines of the file:
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@@
 	(net 78 "MISO")
 	(net 79 "unconnected-(SR_RIGHT1-~{Q7}-Pad7)")
-	(net 80 "unconnected-(SR_RIGHT1-DS-Pad10)")
-	(net 81 "unconnected-(U1-B10-Pad8)")
-	(net 82 "unconnected-(U1-B15-Pad3)")
-	(net 83 "unconnected-(U1-A4-Pad13)")
-	(net 84 "unconnected-(U1-A10-Pad20)")
-	(net 85 "unconnected-(U1-A14-Pad16)")
-	(net 86 "unconnected-(U1-B11-Pad7)")
-	(net 87 "unconnected-(U1-A8-Pad1)")
-	(net 88 "unconnected-(U1-A5-Pad14)")
-	(net 89 "unconnected-(U1-B23-Pad11)")
-	(net 90 "unconnected-(U1-B22-Pad12)")
-	(net 91 "unconnected-(U1-A11-Pad19)")
-	(net 92 "unconnected-(U1-A9-Pad2)")
+	(net 80 "unconnected-(U1-B10-Pad8)")
+	(net 81 "unconnected-(U1-B15-Pad3)")
+	(net 82 "unconnected-(U1-A4-Pad13)")
+	(net 83 "unconnected-(U1-A10-Pad20)")
+	(net 84 "unconnected-(U1-A14-Pad16)")
+	(net 85 "unconnected-(U1-B11-Pad7)")
+	(net 86 "unconnected-(U1-A8-Pad1)")
+	(net 87 "unconnected-(U1-A5-Pad14)")
+	(net 88 "unconnected-(U1-B23-Pad11)")
+	(net 89 "unconnected-(U1-B22-Pad12)")
+	(net 90 "unconnected-(U1-A11-Pad19)")
+	(net 91 "unconnected-(U1-A9-Pad2)")
 	(footprint "keyswitches:Kailh_socket_PG1350_reversible"
 		(layer "F.Cu")
@@
 			(pintype "unspecified")
 		)
-		(model "/home/tong/Documents/kicad/easyeda2kicad/easyeda2kicad.3dshapes/FPC-SMD_12P-P1.00_XYECONN_FPC10-S1.0-12AH2.5.wrl"
+		(model "{$EASYEDA2KICAD}/easyeda2kicad.3dshapes/FPC-SMD_12P-P1.00_XYECONN_FPC10-S1.0-12AH2.5.wrl"
 			(offset
 				(xyz 0 1.65 -0)
@@
 			(layers "F.Cu" "F.Paste" "F.Mask")
 			(roundrect_rratio 0.25)
-			(net 80 "unconnected-(SR_RIGHT1-DS-Pad10)")
+			(net 38 "+3V3")
 			(pinfunction "DS")
-			(pintype "input+no_connect")
+			(pintype "input")
 		)
 		(pad "11" smd roundrect
@@
 			)
 			(remove_unused_layers no)
-			(net 87 "unconnected-(U1-A8-Pad1)")
+			(net 86 "unconnected-(U1-A8-Pad1)")
 			(pinfunction "A8")
 			(pintype "bidirectional+no_connect")
@@
 			)
 			(remove_unused_layers no)
-			(net 92 "unconnected-(U1-A9-Pad2)")
+			(net 91 "unconnected-(U1-A9-Pad2)")
 			(pinfunction "A9")
 			(pintype "bidirectional+no_connect")
@@
 			)
 			(remove_unused_layers no)
-			(net 82 "unconnected-(U1-B15-Pad3)")
+			(net 81 "unconnected-(U1-B15-Pad3)")
 			(pinfunction "B15")
 			(pintype "bidirectional+no_connect")
@@
 			)
 			(remove_unused_layers no)
-			(net 86 "unconnected-(U1-B11-Pad7)")
+			(net 85 "unconnected-(U1-B11-Pad7)")
 			(pinfunction "B11")
 			(pintype "bidirectional+no_connect")
@@
 			)
 			(remove_unused_layers no)
-			(net 81 "unconnected-(U1-B10-Pad8)")
+			(net 80 "unconnected-(U1-B10-Pad8)")
 			(pinfunction "B10")
 			(pintype "bidirectional+no_connect")
@@
 			)
 			(remove_unused_layers no)
-			(net 89 "unconnected-(U1-B23-Pad11)")
+			(net 88 "unconnected-(U1-B23-Pad11)")
 			(pinfunction "B23")
 			(pintype "bidirectional+no_connect")
@@
 			)
 			(remove_unused_layers no)
-			(net 90 "unconnected-(U1-B22-Pad12)")
+			(net 89 "unconnected-(U1-B22-Pad12)")
 			(pinfunction "B22")
 			(pintype "bidirectional+no_connect")
@@
 			)
 			(remove_unused_layers no)
-			(net 83 "unconnected-(U1-A4-Pad13)")
+			(net 82 "unconnected-(U1-A4-Pad13)")
 			(pinfunction "A4")
 			(pintype "bidirectional+no_connect")
@@
 			)
 			(remove_unused_layers no)
-			(net 88 "unconnected-(U1-A5-Pad14)")
+			(net 87 "unconnected-(U1-A5-Pad14)")
 			(pinfunction "A5")
 			(pintype "bidirectional+no_connect")
@@
 			)
 			(remove_unused_layers no)
-			(net 85 "unconnected-(U1-A14-Pad16)")
+			(net 84 "unconnected-(U1-A14-Pad16)")
 			(pinfunction "A14")
 			(pintype "bidirectional+no_connect")
@@
 			)
 			(remove_unused_layers no)
-			(net 91 "unconnected-(U1-A11-Pad19)")
+			(net 90 "unconnected-(U1-A11-Pad19)")
 			(pinfunction "A11")
 			(pintype "bidirectional+no_connect")
@@
 			)
 			(remove_unused_layers no)
-			(net 84 "unconnected-(U1-A10-Pad20)")
+			(net 83 "unconnected-(U1-A10-Pad20)")
 			(pinfunction "A10")
 			(pintype "bidirectional+no_connect")
@@
 			(pintype "unspecified")
 		)
-		(model "/home/tong/Documents/kicad/easyeda2kicad/easyeda2kicad.3dshapes/FPC-SMD_12P-P1.00_XYECONN_FPC10-S1.0-12AH2.5.wrl"
+		(model "${EASYEDA2KICAD}/easyeda2kicad.3dshapes/FPC-SMD_12P-P1.00_XYECONN_FPC10-S1.0-12AH2.5.wrl"
 			(offset
 				(xyz 0 1.65 -0)
